Commit message: uploading to eyantra

File: src/micromouse/urdf/micromouse_robot.urdf (robot description, URDF)
Before this commit: robot micromouse, 1 links, 0 joints
Links:
- added link world
- link base_link: mass None -> 1.0; geometry collision mesh filename=package://micromouse/models/chassis/micromouse.obj; visual mesh filename=package://micromouse/models/chassis/micromouse.obj
Joints:
- added joint joint_name: type fixed, parent world, child base_link, origin xyz=0.0 0.0 0.0 rpy=0.0 0.0 0.0

Commit message: fixed missing libmaze plugin

File: src/micromouse/urdf/micromouse_robot.urdf (robot description, URDF)
Before this commit: robot micromouse, 2 links, 1 joints
Links:
- removed link world
- added link castor_link; collision sphere radius=${radius_castor}; visual sphere radius=${radius_castor}
- link base_link: mass 1.0 -> ${mass_chassis}; geometry collision mesh filename=package://micromouse/models/chassis/micromouse.obj scale=${scale_chassis} ${scale_chassis} ${scale_chassis}; visual mesh filename=package://micromouse/models/chassis/micromouse.obj scale=${scale_chassis} ${scale_chassis} ${scale_chassis}
Joints:
- removed joint joint_name
- added joint castor_wheel: type fixed, parent base_link, child castor_link, origin xyz=0 ${castor_pos_y} -0.006
- added joint left_wheel: type continuous, parent base_link, child left_wheel_link, origin xyz=${wheel_pos_x} ${wheel_pos_y} 0.0 rpy=0 0 0, axis 1 0 0
- added joint right_wheel: type continuous, parent base_link, child right_wheel_link, origin xyz=-${wheel_pos_x} ${wheel_pos_y} 0.0 rpy=0 0 0, axis 1 0 0

Commit message: publishing cmd_vel on micromouse

File: src/micromouse/urdf/micromouse_robot.urdf (robot description, URDF)
Before this commit: robot micromouse, 2 links, 3 joints
Links:
- link base_link: geometry collision box size=0.045 0.004 0.075; visual mesh filename=package://micromouse/models/chassis/micromouse.obj scale=${scale_chassis} ${scale_chassis} ${scale_chassis}
