Commit message: using position controllers

File: src/micromouse/urdf/micromouse_bot.urdf.xacro (robot description, xacro)
@@ -5,6 +5,6 @@
     <xacro:property name="scale_chassis" value="0.25"/>
     <xacro:property name="scale_wheel" value="0.03"/>
-    <xacro:property name="mass_chassis" value="1.2"/>
-    <xacro:property name="mass_wheel" value="0.3"/>
+    <xacro:property name="mass_chassis" value="0.5"/>
+    <xacro:property name="mass_wheel" value="0.01"/>
     <xacro:property name="mass_castor" value="0.2"/>
     <xacro:property name="radius_castor" value="0.005"/>
@@ -14,21 +14,21 @@
     <!-- Import all Gazebo-customization elements, including Gazebo colors -->
     <xacro:include filename="$(find micromouse)/urdf/micromouse_robot.gazebo" />
-    <xacro:macro name="wheel_link" params="name">
+    <xacro:macro name="wheel_link" params="name *origin">
         <link name="${name}_wheel_link">
             <visual>
-                <origin xyz="0 0 0" rpy="0.0 ${rotation_90} 0.0"/>
+                <xacro:insert_block name="origin"/>
                 <geometry>
-                    <mesh filename="package://micromouse/models/wheel/micromouse_wheel.obj" scale="${scale_wheel} ${scale_wheel} ${scale_wheel}"/>
+                    <cylinder radius="0.02" length="0.01"/>
                 </geometry>
             </visual>
             <collision>
-                <origin xyz="0 0 0" rpy="0.0 ${rotation_90} 0.0"/>
+                <xacro:insert_block name="origin"/>
                 <geometry>
-                    <cylinder radius="0.01" length="0.00425"/>
+                    <cylinder radius="0.02" length="0.01"/>
                 </geometry>
             </collision>
             <inertial>
                 <mass value="${mass_wheel}" />
-                <inertia ixx="0.000305" ixy="0.0032" ixz="0.0" iyy="0.009" iyz="8e-6" izz="0.00031" />
+                <inertia ixx="2.3e-06" ixy="0" ixz="0.0" iyy="2.3e-06" iyz="0" izz="4.5e-06" />
             </inertial>
         </link>
@@ -36,22 +36,26 @@
     <link name="base_link">
         <visual>
-            <origin xyz="0.0 0.0 0.0" rpy="${rotation_90} 0.0 0.0"/>
+            <origin xyz="0.0 0.0 0.005" rpy="0.0 0.0 0.0"/>
             <geometry>
-                <mesh filename="package://micromouse/models/chassis/micromouse.obj" scale="${scale_chassis} ${scale_chassis} ${scale_chassis}"/>
+                <box size="0.07 0.07 0.02"/>
             </geometry>
         </visual>
         <collision>
-            <origin xyz="0.0 0.0 0.0" rpy="${rotation_90} 0.0 0.0"/>
+            <origin xyz="0.0 0.0 0.005" rpy="0.0 0.0 0.0"/>
             <geometry>
-                <box size="0.045 0.004 0.075"/>
+                <box size="0.07 0.07 0.02"/>
             </geometry>
         </collision>
         <inertial>
             <mass value="${mass_chassis}" />
-            <inertia ixx="0.012" ixy="1.5e-6" ixz="0.0" iyy="0.01" iyz="0.0" izz="0.12" />
+            <inertia ixx="0.00022083" ixy="0.0" ixz="0.0" iyy="0.00022083" iyz="0.0" izz="0.00040833" />
         </inertial>
     </link>
-    <xacro:wheel_link name="left"/>
-    <xacro:wheel_link name="right"/>
+    <xacro:wheel_link name="left">
+        <origin xyz="0.02 0.0 0.0" rpy="0.0 ${rotation_90} 0.0"/>
+    </xacro:wheel_link>
+    <xacro:wheel_link name="right">
+        <origin xyz="-0.02 0.0 0.0" rpy="0.0 ${rotation_90} 0.0"/>
+    </xacro:wheel_link>
     <link name="castor_link">
         <visual>
@@ -65,5 +69,5 @@
             </geometry>
             <inertial>
-                <origin xyz="0.0 0.0 0.0" rpy="0.0 0.0 0.0"/>
+                <origin xyz="0.0 0.03 -0.02" rpy="0.0 0.0 0.0"/>
                 <mass value="${mass_castor}"/>
                 <inertia ixx="0.002" ixy="0.0" ixz="0.0" iyy="0.002" iyz="0.0" izz="0.002"/>
@@ -76,5 +80,6 @@
         <axis xyz="1 0 0"/>
         <origin xyz="${wheel_pos_x} ${wheel_pos_y} 0.0" rpy="0 0 0"/>
-        <limit effort="1000.0" velocity="100.0"/>
+        <limit effort="-1" velocity="100.0"/>
+        <dynamics damping="0.01" friction="0.0"/>
     </joint>
     <joint name="right_wheel" type="continuous">
@@ -83,5 +88,6 @@
         <axis xyz="1 0 0"/>
         <origin xyz="-${wheel_pos_x} ${wheel_pos_y} 0.0" rpy="0 0 0"/>
-        <limit effort="1000.0" velocity="100.0"/>
+        <limit effort="-1" velocity="100.0"/>
+        <dynamics damping="0.01" friction="0.0"/>
     </joint>
     <joint name="castor_wheel" type="fixed">

Commit message: trying to make a mouse in urdf

File: src/micromouse/urdf/micromouse_bot.urdf.xacro (robot description, xacro)
@@ -1,119 +1,123 @@
 <?xml version="1.0"?>
-<robot name="micromouse" xmlns:xacro="http://www.ros.org/wiki/xacro">
-    <!-- Constants for robot -->
-    <xacro:property name="rotation_90" value="1.57079632679"/>
-    <xacro:property name="scale_chassis" value="0.25"/>
-    <xacro:property name="scale_wheel" value="0.03"/>
-    <xacro:property name="mass_chassis" value="0.5"/>
-    <xacro:property name="mass_wheel" value="0.01"/>
-    <xacro:property name="mass_castor" value="0.2"/>
-    <xacro:property name="radius_castor" value="0.005"/>
-    <xacro:property name="wheel_pos_x" value="0.026"/>
-    <xacro:property name="wheel_pos_y" value="-0.016"/>
-    <xacro:property name="castor_pos_y" value="0.025"/>
-    <!-- Import all Gazebo-customization elements, including Gazebo colors -->
-    <xacro:include filename="$(find micromouse)/urdf/micromouse_robot.gazebo" />
-    <xacro:macro name="wheel_link" params="name *origin">
-        <link name="${name}_wheel_link">
-            <visual>
-                <xacro:insert_block name="origin"/>
-                <geometry>
-                    <cylinder radius="0.02" length="0.01"/>
-                </geometry>
-            </visual>
-            <collision>
-                <xacro:insert_block name="origin"/>
-                <geometry>
-                    <cylinder radius="0.02" length="0.01"/>
-                </geometry>
-            </collision>
-            <inertial>
-                <mass value="${mass_wheel}" />
-                <inertia ixx="2.3e-06" ixy="0" ixz="0.0" iyy="2.3e-06" iyz="0" izz="4.5e-06" />
-            </inertial>
-        </link>
+<robot name="micromouse" xmlns:xacro="https://www.ros.org/wiki/xacro">
+    <material name="body_texture">
+        <color rgba="0.2 0.4 0.2 1.0"/>
+    </material>
+    <material name="black">
+        <color rgba="0.0 0.0 0.0 1.0"/>
+    </material>
+    <xacro:property name="rotate_90" value="1.57079632679"/>
+    <xacro:property name="head_radius" value="0.025"/>
+    <xacro:property name="body_radius" value="0.020"/>
+    <xacro:property name="body_length" value="0.07"/>
+    <xacro:macro name="default_inertial">
+        <inertial>
+            <mass value="0.001" />
+            <inertia ixx="1e-06" ixy="0.0" ixz="0.0" iyy="1e-06" iyz="0.0" izz="1e-06" />
+        </inertial>
     </xacro:macro>
-    <link name="base_link">
+    <link name="base_link"/>
+    <link name="mouse_body_link">
+        <inertial>
+            <origin xyz="0.0 0.0 0.0" rpy="0.0 0.0 0.0"/>
+            <mass value="0.5"/>
+            <inertia ixx="0.00022083" ixy="0.0" ixz="0.0" iyy="0.00022083" iyz="0.0" izz="0.00040833"/>
+        </inertial>
+        <visual name="body">
+            <origin xyz="0.0 0.0 0.0" rpy="${rotate_90} 0.0 0.0"/>
+            <geometry>
+                <cylinder radius="${body_radius}" length="${body_length}"/>
+            </geometry>
+            <material name="body_texture"/>
+        </visual>
+        <collision name="body">
+            <origin xyz="0.0 0.0 0.0" rpy="${rotate_90} 0.0 0.0"/>
+            <geometry>
+                <cylinder radius="${body_radius}" length="${body_length}"/>
+            </geometry>
+        </collision>
+        <visual name="left_base">
+            <geometry>
+                <box size="0.005 0.06 0.02"/>
+            </geometry>
+            <material name="body_texture"/>
+        </visual>
+        <collision name="left_base">
+            <geometry>
+                <box size="0.005 0.06 0.02"/>
+            </geometry>
+            <material name="body_texture"/>
+        </collision>
+    </link>
+    <joint name="dummy_joint" type="fixed">
+        <parent link="base_link"/>
+        <child link="mouse_body_link"/>
+    </joint>
+    <link name="mouse_head_link">
+        <inertial>
+            <origin xyz="0.0 0.0 0.0" rpy="0.0 0.0 0.0"/>
+            <mass value="0.2"/>
+            <inertia ixx="0.00015" ixy="0.0" ixz="0.0" iyy="0.00015" iyz="0.0" izz="0.00015"/>
+        </inertial>
+        <visual name="head">
+            <origin xyz="0.0 ${body_length/2} 0.0" rpy="0.0 0.0 0.0"/>
+            <geometry>
+                <sphere radius="${head_radius}"/>
+            </geometry>
+            <material name="body_texture"/>
+        </visual>
+        <collision name="head">
+            <origin xyz="0.0 ${body_length/2} 0.0" rpy="0.0 0.0 0.0"/>
+            <geometry>
+                <sphere radius="${head_radius}"/>
+            </geometry>
+        </collision>
+    </link>
+    <joint name="mouse_head_joint" type="revolute">
+        <parent link="mouse_body_link"/>
+        <child link="mouse_head_link"/>
+        <axis xyz="0 0 1"/>
+        <limit lower="-${rotate_90/8}" upper="${rotate_90/8}" velocity="5.0" effort="10.0"/>
+        <origin xyz="0 0 0" rpy="0 0 0"/>
+    </joint>
+    <link name="mouse_left_eye_link">
         <visual>
-            <origin xyz="0.0 0.0 0.005" rpy="0.0 0.0 0.0"/>
+            <origin xyz="-0.01 0.05 0.01"/>
             <geometry>
-                <box size="0.07 0.07 0.02"/>
+                <sphere radius="0.001"/>
             </geometry>
+            <material name="black"/>
         </visual>
         <collision>
-            <origin xyz="0.0 0.0 0.005" rpy="0.0 0.0 0.0"/>
+            <origin xyz="-0.01 0.05 0.01"/>
             <geometry>
-                <box size="0.07 0.07 0.02"/>
+                <sphere radius="0.001"/>
             </geometry>
         </collision>
-        <inertial>
-            <mass value="${mass_chassis}" />
-            <inertia ixx="0.00022083" ixy="0.0" ixz="0.0" iyy="0.00022083" iyz="0.0" izz="0.00040833" />
-        </inertial>
+        <xacro:default_inertial/>
     </link>
-    <xacro:wheel_link name="left">
-        <origin xyz="0.02 0.0 0.0" rpy="0.0 ${rotation_90} 0.0"/>
-    </xacro:wheel_link>
-    <xacro:wheel_link name="right">
-        <origin xyz="-0.02 0.0 0.0" rpy="0.0 ${rotation_90} 0.0"/>
-    </xacro:wheel_link>
-    <link name="castor_link">
+    <joint name="left_eye_joint" type="fixed">
+        <parent link="mouse_head_link"/>
+        <child link="mouse_left_eye_link"/>
+    </joint>
+    <link name="mouse_right_eye_link">
         <visual>
+            <origin xyz="0.01 0.05 0.01"/>
             <geometry>
-                <sphere radius="${radius_castor}"/>
+                <sphere radius="0.001"/>
             </geometry>
+            <material name="black"/>
         </visual>
         <collision>
+            <origin xyz="0.01 0.05 0.01"/>
             <geometry>
-                <sphere radius="${radius_castor}"/>
+                <sphere radius="0.001"/>
             </geometry>
-            <inertial>
-                <origin xyz="0.0 0.03 -0.02" rpy="0.0 0.0 0.0"/>
-                <mass value="${mass_castor}"/>
-                <inertia ixx="0.002" ixy="0.0" ixz="0.0" iyy="0.002" iyz="0.0" izz="0.002"/>
-            </inertial>
         </collision>
+        <xacro:default_inertial/>
     </link>
-    <joint name="left_wheel" type="continuous">
-        <parent link="base_link"/>
-        <child link="left_wheel_link"/>
-        <axis xyz="1 0 0"/>
-        <origin xyz="${wheel_pos_x} ${wheel_pos_y} 0.0" rpy="0 0 0"/>
-        <limit effort="-1" velocity="100.0"/>
-        <dynamics damping="0.01" friction="0.0"/>
+    <joint name="right_eye_joint" type="fixed">
+        <parent link="mouse_head_link"/>
+        <child link="mouse_right_eye_link"/>
     </joint>
-    <joint name="right_wheel" type="continuous">
-        <parent link="base_link"/>
-        <child link="right_wheel_link"/>
-        <axis xyz="1 0 0"/>
-        <origin xyz="-${wheel_pos_x} ${wheel_pos_y} 0.0" rpy="0 0 0"/>
-        <limit effort="-1" velocity="100.0"/>
-        <dynamics damping="0.01" friction="0.0"/>
-    </joint>
-    <joint name="castor_wheel" type="fixed">
-        <parent link="base_link"/>
-        <child link="castor_link"/>
-        <origin xyz="0 ${castor_pos_y} -0.006"/>
-    </joint>
-    <!-- Transmission is important to link the joints and the controller -->
-    <transmission name="left_wheel_trans">
-        <type>transmission_interface/SimpleTransmission</type>
-        <joint name="left_wheel">
-            <hardwareInterface>hardware_interface/VelocityJointInterface</hardwareInterface>
-        </joint>
-        <actuator name="left_wheel_motor">
-            <hardwareInterface>EffortJointInterface</hardwareInterface>
-            <mechanicalReduction>1</mechanicalReduction>
-        </actuator>
-    </transmission>
-    <transmission name="right_wheel_trans">
-        <type>transmission_interface/SimpleTransmission</type>
-        <joint name="right_wheel">
-            <hardwareInterface>hardware_interface/VelocityJointInterface</hardwareInterface>
-        </joint>
-        <actuator name="right_wheel_motor">
-            <hardwareInterface>EffortJointInterface</hardwareInterface>
-            <mechanicalReduction>1</mechanicalReduction>
-        </actuator>
-    </transmission>
 </robot>

File: src/micromouse/urdf/micromouse_robot.urdf (robot description, URDF)
Before this commit: robot micromouse, 2 links, 3 joints
Links:
- added link dummy
Joints:
- added joint dummy_joint: type fixed, parent dummy, child base_link
