Commit message: deleting unnecessary files

File: src/micromouse/urdf/micromouse_bot.urdf.xacro (robot description, xacro)
@@ -1,4 +1,6 @@
 <?xml version="1.0"?>
 <robot name="micromouse" xmlns:xacro="https://www.ros.org/wiki/xacro">
+    <!-- Import all Gazebo-customization elements, including Gazebo colors -->
+    <xacro:include filename="$(find micromouse)/urdf/micromouse_bot.gazebo" />
     <material name="body_texture">
         <color rgba="0.2 0.4 0.2 1.0"/>
@@ -7,8 +9,8 @@
         <color rgba="0.0 0.0 0.0 1.0"/>
     </material>
-    <xacro:property name="rotate_90" value="1.57079632679"/>
+    <xacro:property name="rotate" value="1.57079632679"/>
     <xacro:property name="head_radius" value="0.025"/>
     <xacro:property name="body_radius" value="0.020"/>
-    <xacro:property name="body_length" value="0.07"/>
+    <xacro:property name="body_length" value="0.05"/>
     <xacro:macro name="default_inertial">
         <inertial>
@@ -24,6 +26,6 @@
             <inertia ixx="0.00022083" ixy="0.0" ixz="0.0" iyy="0.00022083" iyz="0.0" izz="0.00040833"/>
         </inertial>
-        <visual name="body">
-            <origin xyz="0.0 0.0 0.0" rpy="${rotate_90} 0.0 0.0"/>
+        <visual>
+            <origin xyz="0.0 0.0 0.0" rpy="${rotate} 0.0 0.0"/>
             <geometry>
                 <cylinder radius="${body_radius}" length="${body_length}"/>
@@ -32,20 +34,21 @@
         </visual>
         <collision name="body">
-            <origin xyz="0.0 0.0 0.0" rpy="${rotate_90} 0.0 0.0"/>
+            <origin xyz="0.0 0.0 0.0" rpy="${rotate} 0.0 0.0"/>
             <geometry>
                 <cylinder radius="${body_radius}" length="${body_length}"/>
             </geometry>
         </collision>
-        <visual name="left_base">
-            <geometry>
-                <box size="0.005 0.06 0.02"/>
+        <visual>
+            <origin xyz="0.0 ${body_length/2} 0.0"/>
+            <geometry>
+                <sphere radius="${body_radius}"/>
             </geometry>
             <material name="body_texture"/>
         </visual>
-        <collision name="left_base">
-            <geometry>
-                <box size="0.005 0.06 0.02"/>
-            </geometry>
-            <material name="body_texture"/>
+        <collision>
+            <origin xyz="0.0 ${body_length/2} 0.0"/>
+            <geometry>
+                <sphere radius="${body_radius}"/>
+            </geometry>
         </collision>
     </link>
@@ -55,11 +58,7 @@
     </joint>
     <link name="mouse_head_link">
-        <inertial>
-            <origin xyz="0.0 0.0 0.0" rpy="0.0 0.0 0.0"/>
-            <mass value="0.2"/>
-            <inertia ixx="0.00015" ixy="0.0" ixz="0.0" iyy="0.00015" iyz="0.0" izz="0.00015"/>
-        </inertial>
-        <visual name="head">
-            <origin xyz="0.0 ${body_length/2} 0.0" rpy="0.0 0.0 0.0"/>
+        <xacro:default_inertial/>
+        <visual>
+            <origin xyz="0.0 -${body_length/2} 0.0" rpy="0.0 0.0 0.0"/>
             <geometry>
                 <sphere radius="${head_radius}"/>
@@ -67,6 +66,6 @@
             <material name="body_texture"/>
         </visual>
-        <collision name="head">
-            <origin xyz="0.0 ${body_length/2} 0.0" rpy="0.0 0.0 0.0"/>
+        <collision>
+            <origin xyz="0.0 -${body_length/2} 0.0" rpy="0.0 0.0 0.0"/>
             <geometry>
                 <sphere radius="${head_radius}"/>
@@ -74,23 +73,22 @@
         </collision>
     </link>
-    <joint name="mouse_head_joint" type="revolute">
+    <joint name="mouse_head_joint" type="fixed">
         <parent link="mouse_body_link"/>
         <child link="mouse_head_link"/>
-        <axis xyz="0 0 1"/>
-        <limit lower="-${rotate_90/8}" upper="${rotate_90/8}" velocity="5.0" effort="10.0"/>
-        <origin xyz="0 0 0" rpy="0 0 0"/>
+        <!-- <axis xyz="0 0 1"/> -->
+        <!-- <limit lower="-${rotate/8}" upper="${rotate/8}" velocity="5.0" effort="10.0"/> -->
     </joint>
     <link name="mouse_left_eye_link">
         <visual>
-            <origin xyz="-0.01 0.05 0.01"/>
-            <geometry>
-                <sphere radius="0.001"/>
-            </geometry>
-            <material name="black"/>
-        </visual>
-        <collision>
-            <origin xyz="-0.01 0.05 0.01"/>
-            <geometry>
-                <sphere radius="0.001"/>
+            <origin xyz="-0.01 -${body_length/2+head_radius-0.005} 0.01"/>
+            <geometry>
+                <sphere radius="0.004"/>
+            </geometry>
+            <material name="black"/>
+        </visual>
+        <collision>
+            <origin xyz="-0.01 -${body_length/2+head_radius-0.005} 0.01"/>
+            <geometry>
+                <sphere radius="0.004"/>
             </geometry>
         </collision>
@@ -103,14 +101,14 @@
     <link name="mouse_right_eye_link">
         <visual>
-            <origin xyz="0.01 0.05 0.01"/>
-            <geometry>
-                <sphere radius="0.001"/>
-            </geometry>
-            <material name="black"/>
-        </visual>
-        <collision>
-            <origin xyz="0.01 0.05 0.01"/>
-            <geometry>
-                <sphere radius="0.001"/>
+            <origin xyz="0.01 -${body_length/2+head_radius-0.005} 0.01"/>
+            <geometry>
+                <sphere radius="0.004"/>
+            </geometry>
+            <material name="black"/>
+        </visual>
+        <collision>
+            <origin xyz="0.01 -${body_length/2+head_radius-0.005} 0.01"/>
+            <geometry>
+                <sphere radius="0.004"/>
             </geometry>
         </collision>
@@ -121,3 +119,98 @@
         <child link="mouse_right_eye_link"/>
     </joint>
+    <link name="mouse_nose_link">
+        <visual>
+            <geometry>
+                <cylinder radius="0.006" length="0.0055"/>
+            </geometry>
+            <material name="black"/>
+        </visual>
+        <collision>
+            <geometry>
+                <cylinder radius="0.006" length="0.0055"/>
+            </geometry>
+        </collision>
+        <xacro:default_inertial/>
+    </link>
+    <joint name="mouse_nose_joint" type="fixed">
+        <parent link="mouse_head_link"/>
+        <child link="mouse_nose_link"/>
+        <origin xyz="0.0 -${body_length/2+head_radius-0.005} -0.01" rpy="${2*rotate} 0.0 0"/>
+    </joint>
+    <link name="right_wheel_link">
+        <inertial>
+            <origin xyz="0.0 0.0 0.0" rpy="0.0 ${rotate} 0.0"/>
+            <mass value="0.2"/>
+            <inertia ixx="2.3e-06" ixy="0.0" ixz="0.0" iyy="2.3e-06" iyz="0.0" izz="4.5e-06"/>
+        </inertial>
+        <visual>
+            <origin xyz="0.0 0.0 0.0" rpy="0.0 ${rotate} 0.0"/>
+            <geometry>
+                <cylinder radius="0.02" length="0.01"/>
+            </geometry>
+            <material name="black"/>
+        </visual>
+        <collision>
+            <origin xyz="0.0 0.0 0.0" rpy="0.0 ${rotate} 0.0"/>
+            <geometry>
+                <cylinder radius="0.02" length="0.01"/>
+            </geometry>
+        </collision>
+    </link>
+    <joint name="right_wheel_joint" type="continuous">
+        <parent link="mouse_body_link"/>
+        <child link="right_wheel_link"/>
+        <axis xyz="1 0 0"/>
+        <origin xyz="-0.025  0.02 -0.005" rpy="0 0 0"/>
+        <limit effort="-1" velocity="100"/>
+        <joint_properties damping="0.01" friction="0.0" />
+    </joint>
+    <transmission name="right_wheel_trans">
+        <type>transmission_interface/SimpleTransmission</type>
+        <joint name="right_wheel_joint">
+            <hardwareInterface>hardware_interface/VelocityJointInterface</hardwareInterface>
+        </joint>
+        <actuator name="right_wheel_motor">
+            <hardwareInterface>hardware_interface/VelocityJointInterface</hardwareInterface>
+            <mechanicalReduction>7</mechanicalReduction>
+        </actuator>
+    </transmission>
+    <link name="left_wheel_link">
+        <inertial>
+            <origin xyz="0.0 0.0 0.0" rpy="0.0 ${rotate} 0.0"/>
+            <mass value="0.2"/>
+            <inertia ixx="2.3e-06" ixy="0.0" ixz="0.0" iyy="2.3e-06" iyz="0.0" izz="4.5e-06"/>
+        </inertial>
+        <visual>
+            <origin xyz="0.0 0.0 0.0" rpy="0.0 ${rotate} 0.0"/>
+            <geometry>
+                <cylinder radius="0.02" length="0.01"/>
+            </geometry>
+            <material name="black"/>
+        </visual>
+        <collision>
+            <origin xyz="0.0 0.0 0.0" rpy="0.0 ${rotate} 0.0"/>
+            <geometry>
+                <cylinder radius="0.02" length="0.01"/>
+            </geometry>
+        </collision>
+    </link>
+    <joint name="left_wheel_joint" type="continuous">
+        <parent link="mouse_body_link"/>
+        <child link="left_wheel_link"/>
+        <axis xyz="1 0 0"/>
+        <origin xyz="0.025  0.02 -0.005" rpy="0 0 0"/>
+        <limit effort="-1" velocity="100"/>
+        <joint_properties damping="0.01" friction="0.0" />
+    </joint>
+    <transmission name="left_wheel_trans">
+        <type>transmission_interface/SimpleTransmission</type>
+        <joint name="left_wheel_joint">
+            <hardwareInterface>hardware_interface/VelocityJointInterface</hardwareInterface>
+        </joint>
+        <actuator name="left_wheel_motor">
+            <hardwareInterface>hardware_interface/VelocityJointInterface</hardwareInterface>
+            <mechanicalReduction>7</mechanicalReduction>
+        </actuator>
+    </transmission>
 </robot>

Commit message: Added launch, worlds

File: src/micromouse/urdf/micromouse_bot.urdf.xacro (robot description, xacro)
@@ -3,5 +3,5 @@
     <!-- Import all Gazebo-customization elements, including Gazebo colors -->
     <xacro:include filename="$(find micromouse)/urdf/micromouse_bot.gazebo" />
-    <material name="body_texture">
+    <material name="green">
         <color rgba="0.2 0.4 0.2 1.0"/>
     </material>
@@ -19,5 +19,4 @@
         </inertial>
     </xacro:macro>
-    <link name="base_link"/>
     <link name="mouse_body_link">
         <inertial>
@@ -31,5 +30,5 @@
                 <cylinder radius="${body_radius}" length="${body_length}"/>
             </geometry>
-            <material name="body_texture"/>
+            <material name="green"/>
         </visual>
         <collision name="body">
@@ -44,7 +43,7 @@
                 <sphere radius="${body_radius}"/>
             </geometry>
-            <material name="body_texture"/>
+            <material name="green"/>
         </visual>
-        <collision>
+        <collision name="butt">
             <origin xyz="0.0 ${body_length/2} 0.0"/>
             <geometry>
@@ -52,11 +51,4 @@
             </geometry>
         </collision>
-    </link>
-    <joint name="dummy_joint" type="fixed">
-        <parent link="base_link"/>
-        <child link="mouse_body_link"/>
-    </joint>
-    <link name="mouse_head_link">
-        <xacro:default_inertial/>
         <visual>
             <origin xyz="0.0 -${body_length/2} 0.0" rpy="0.0 0.0 0.0"/>
@@ -64,5 +56,5 @@
                 <sphere radius="${head_radius}"/>
             </geometry>
-            <material name="body_texture"/>
+            <material name="green"/>
         </visual>
         <collision>
@@ -72,13 +64,5 @@
             </geometry>
         </collision>
-    </link>
-    <joint name="mouse_head_joint" type="fixed">
-        <parent link="mouse_body_link"/>
-        <child link="mouse_head_link"/>
-        <!-- <axis xyz="0 0 1"/> -->
-        <!-- <limit lower="-${rotate/8}" upper="${rotate/8}" velocity="5.0" effort="10.0"/> -->
-    </joint>
-    <link name="mouse_left_eye_link">
-        <visual>
+        <visual name="left_eye">
             <origin xyz="-0.01 -${body_length/2+head_radius-0.005} 0.01"/>
             <geometry>
@@ -93,12 +77,5 @@
             </geometry>
         </collision>
-        <xacro:default_inertial/>
-    </link>
-    <joint name="left_eye_joint" type="fixed">
-        <parent link="mouse_head_link"/>
-        <child link="mouse_left_eye_link"/>
-    </joint>
-    <link name="mouse_right_eye_link">
-        <visual>
+        <visual name="right_eye">
             <origin xyz="0.01 -${body_length/2+head_radius-0.005} 0.01"/>
             <geometry>
@@ -113,12 +90,6 @@
             </geometry>
         </collision>
-        <xacro:default_inertial/>
-    </link>
-    <joint name="right_eye_joint" type="fixed">
-        <parent link="mouse_head_link"/>
-        <child link="mouse_right_eye_link"/>
-    </joint>
-    <link name="mouse_nose_link">
-        <visual>
+        <visual name="nose">
+            <origin xyz="0.0 -${body_length/2+head_radius-0.005} -0.01" rpy="${2*rotate} 0.0 0"/>
             <geometry>
                 <cylinder radius="0.006" length="0.0055"/>
@@ -127,15 +98,10 @@
         </visual>
         <collision>
+            <origin xyz="0.0 -${body_length/2+head_radius-0.005} -0.01" rpy="${2*rotate} 0.0 0"/>
             <geometry>
                 <cylinder radius="0.006" length="0.0055"/>
             </geometry>
         </collision>
-        <xacro:default_inertial/>
     </link>
-    <joint name="mouse_nose_joint" type="fixed">
-        <parent link="mouse_head_link"/>
-        <child link="mouse_nose_link"/>
-        <origin xyz="0.0 -${body_length/2+head_radius-0.005} -0.01" rpy="${2*rotate} 0.0 0"/>
-    </joint>
     <link name="right_wheel_link">
         <inertial>
