Commit message: added solution to bowling game

File: src/pkg_gazebo/urdf/bowling_ball_bot.urdf.xacro (robot description, xacro)
@@ -1,8 +1,9 @@
 <?xml version="1.0"?>
 <robot name="bowling_ball" xmlns:xacro="http://ros.org/wiki/xacro">
+    <!-- Import all Gazebo-customization elements, including Gazebo colors -->
+    <xacro:include filename="$(find pkg_gazebo)/urdf/bowling_ball_bot.gazebo" />
     <!-- Constants for robot -->
-    <xacro:property name="radius" value="0.11"/>
+    <xacro:property name="radius" value="0.2"/>
     <xacro:property name="mass" value="8.0"/>
-    <xacro:property name="link_name" value="dummy"/>
     <material name="gloss_black">
         <color rgba="${37/255} ${35/255} ${36/255} 1"/>
@@ -11,5 +12,5 @@
         <visual>
             <geometry>
-                <sphere radius="${radius}"/>
+                <sphere radius="0.2"/>
             </geometry>
             <material name="gloss_black"/>
@@ -18,10 +19,10 @@
         <collision>
             <geometry>
-                <sphere radius="${radius}"/>
+                <sphere radius="0.2"/>
             </geometry>
             <origin xyz="0.0 0.0 0.0" rpy="0.0 0.0 0.0"/>
         </collision>
         <inertial>
-            <mass value="${mass}" />
+            <mass value="8.0" />
             <inertia ixx="0.03872" ixy="0.004" ixz="0.005" iyy="0.03872" iyz="0.003" izz="0.03872" />
         </inertial>
@@ -29,24 +30,24 @@
     <link name="dummy">
         <inertial>
-            <mass value="0.025" />
-            <inertia ixx="5.8083e-4" ixy="0" ixz="0" iyy="3.0833e-5" iyz="0" izz="5.9083e-4" />
+            <mass value="1e-04" />
+            <inertia ixx="1e-06" ixy="0" ixz="0" iyy="1e-06" iyz="0" izz="1e-06" />
         </inertial>
     </link>
     <link name="rotx_link">
         <inertial>
-            <mass value="0.025" />
-            <inertia ixx="5.8083e-4" ixy="0" ixz="0" iyy="3.0833e-5" iyz="0" izz="5.9083e-4" />
+            <mass value="1e-04" />
+            <inertia ixx="1e-06" ixy="0" ixz="0" iyy="1e-06" iyz="0" izz="1e-06" />
         </inertial>
     </link>
     <link name="roty_link">
         <inertial>
-            <mass value="0.025" />
-            <inertia ixx="5.8083e-4" ixy="0" ixz="0" iyy="3.0833e-5" iyz="0" izz="5.9083e-4" />
+            <mass value="1e-04" />
+            <inertia ixx="1e-06" ixy="0" ixz="0" iyy="1e-06" iyz="0" izz="1e-06" />
         </inertial>
     </link>
     <link name="rotz_link">
         <inertial>
-            <mass value="0.025" />
-            <inertia ixx="5.8083e-4" ixy="0" ixz="0" iyy="3.0833e-5" iyz="0" izz="5.9083e-4" />
+            <mass value="1e-04" />
+            <inertia ixx="1e-06" ixy="0" ixz="0" iyy="1e-06" iyz="0" izz="1e-06" />
         </inertial>
     </link>
@@ -70,87 +71,33 @@
         <child link="dummy"/>
     </joint>
-    <!-- Gazebo Plugin for ROS Control -->
-    <gazebo>
-        <plugin name="gazebo_ros_control" filename="libgazebo_ros_control.so">
-            <robotNamespace>/</robotNamespace>
-        </plugin>
-    </gazebo>
-    <gazebo reference="base_link">
-        <visual name="gazebo_visual">
-            <material>
-                <lighting>1</lighting>
-                <script>
-                    <uri>file://media/materials/scripts/gazebo.material</uri>
-                    <name>Gazebo/Black</name>
-                </script>
-            <shader type='pixel'>
-                <normal_map>__default__</normal_map>
-            </shader>
-            <ambient>0.3 0.3 0.3 1</ambient>
-            <diffuse>0.7 0.7 0.7 1</diffuse>
-            <specular>0.14509803921 0.13725490196 0.14117647058 1</specular>
-            <emissive>0 0 0 1</emissive>
-            </material>
-        </visual>
-        <collision name="gazebo_collision">
-            <surface>
-                <friction>
-                    <ode>
-                        <mu>0.2</mu>
-                        <mu2>0.2</mu2>
-                    </ode>
-                </friction>
-            </surface>
-        </collision>
-    </gazebo>
-    <gazebo reference="${link_name}">
-        <sensor name="${link_name}_camera" type="depth">
-            <update_rate>20</update_rate>
-            <camera>
-                <horizontal_fov>1.047198</horizontal_fov>
-                <image>
-                    <width>640</width>
-                    <height>480</height>
-                    <format>R8G8B8</format>
-                </image>
-                <clip>
-                    <near>0.05</near>
-                    <far>3</far>
-                </clip>
-            </camera>
-        <plugin name="${link_name}_controller" filename="libgazebo_ros_openni_kinect.so">
-            <baseline>0.2</baseline>
-            <alwaysOn>true</alwaysOn>
-            <updateRate>1.0</updateRate>
-            <cameraName>${camera_name}_ir</cameraName>
-            <imageTopicName>/${camera_name}/color/image_raw</imageTopicName>
-            <cameraInfoTopicName>/${camera_name}/color/camera_info</cameraInfoTopicName>
-            <depthImageTopicName>/${camera_name}/depth/image_raw</depthImageTopicName>
-            <depthImageInfoTopicName>/${camera_name}/depth/camera_info</depthImageInfoTopicName>
-            <pointCloudTopicName>/${camera_name}/depth/points</pointCloudTopicName>
-            <frameName>${frame_name}</frameName>
-            <pointCloudCutoff>0.5</pointCloudCutoff>
-            <pointCloudCutoffMax>3.0</pointCloudCutoffMax>
-            <distortionK1>0.00000001</distortionK1>
-            <distortionK2>0.00000001</distortionK2>
-            <distortionK3>0.00000001</distortionK3>
-            <distortionT1>0.00000001</distortionT1>
-            <distortionT2>0.00000001</distortionT2>
-            <CxPrime>0</CxPrime>
-            <Cx>0</Cx>
-            <Cy>0</Cy>
-            <focalLength>0</focalLength>
-            <hackBaseline>0</hackBaseline>
-        </plugin>
-        </sensor>
-    </gazebo>
     <!-- This block provides movement of ball bot -->
     <transmission name="move_x">
         <type>transmission_interface/SimpleTransmission</type>
-        <actuator name="$move_x">
+        <actuator name="move_x">
             <mechanicalReduction>1</mechanicalReduction>
+            <hardwareInterface>EffortJointInterface</hardwareInterface>
         </actuator>
         <joint name="rotate_x">
-            <hardwareInterface>hardware_interface/VelocityJointInterface</hardwareInterface>
+            <hardwareInterface>hardware_interface/EffortJointInterface</hardwareInterface>
+        </joint>
+    </transmission>
+    <transmission name="move_y">
+        <type>transmission_interface/SimpleTransmission</type>
+        <actuator name="move_y">
+            <mechanicalReduction>1</mechanicalReduction>
+            <hardwareInterface>EffortJointInterface</hardwareInterface>
+        </actuator>
+        <joint name="rotate_y">
+            <hardwareInterface>hardware_interface/EffortJointInterface</hardwareInterface>
+        </joint>
+    </transmission>
+    <transmission name="move_z">
+        <type>transmission_interface/SimpleTransmission</type>
+        <actuator name="move_z">
+            <mechanicalReduction>1</mechanicalReduction>
+            <hardwareInterface>EffortJointInterface</hardwareInterface>
+        </actuator>
+        <joint name="rotate_z">
+            <hardwareInterface>hardware_interface/EffortJointInterface</hardwareInterface>
         </joint>
     </transmission>
